Commit message: Added container links to robot model

File: urdf/suii_description.urdf.xacro (robot description, xacro)
@@ -10,7 +10,22 @@
     <origin xyz="0.0 0.0 0.0207767" rpy="0 0 ${-pi/2.0}" />
   </joint>
+  <link name="container_1"/>
+  <link name="container_2"/>
+  <link name="container_3"/>
+  <joint name="containter_1_mount" type="fixed">
+    <parent link="ur3/base" />
+    <child link="container_1" />
+    <origin xyz="-0.116716759233 0.243108042094 0.096870664897" rpy="0.046614 -0.0489053 2.1264592" />
+  </joint>
+  <joint name="containter_2_mount" type="fixed">
+    <parent link="ur3/base" />
+    <child link="container_2" />
+    <origin xyz="0.0160084875755 0.274635895309 0.0989370326304" rpy="0.023152 -0.0237985 1.604636" />
+  </joint>
+  <joint name="containter_3_mount" type="fixed">
+    <parent link="ur3/base" />
+    <child link="container_3" />
+    <origin xyz="0.142679287389 0.228439321043 0.0976393529311" rpy="0.0169812 0.0146731 1.0212226" />
+  </joint>
   <xacro:suii_base/>
-  <!--<xacro:ur_robot parent="arm_placeholder" prefix="ur3/" joint_limited="false">
-    <origin xyz="0.0 0.0 0.0207767" rpy="0.0 0.0 -1.5707963267949" />
-    </xacro:ur_robot>-->
 </robot>

Commit message: Added object picking from tf

File: urdf/suii_description.urdf.xacro (robot description, xacro)
@@ -13,4 +13,5 @@
   <link name="container_2"/>
   <link name="container_3"/>
+  <link name="gripper"/>
   <joint name="containter_1_mount" type="fixed">
     <parent link="ur3/base" />
@@ -28,4 +29,9 @@
     <origin xyz="0.142679287389 0.228439321043 0.0976393529311" rpy="0.0169812 0.0146731 1.0212226" />
   </joint>
+  <joint name="gripper_joint" type="fixed">
+    <parent link="ur3/tool0" />
+    <child link="gripper" />
+    <origin xyz="0 0 0.2" rpy="${pi} 0 0" />
+  </joint>
   <xacro:suii_base/>
 </robot>
